Commit message: minor improvements

File: system/controller/simulation/p3dx/pioneer3dx.urdf (robot description, URDF)
Before this commit: robot pioneer3dx, 11 links, 10 joints
Links:
- link base_link: geometry collision box size=0.35 0.25 0.14; visual mesh filename=meshes/chassis.stl
- link center_hubcap: geometry collision box size=0.00001 0.00001 0.00001; visual mesh filename=meshes/center_hubcap.stl
- link center_wheel: geometry collision cylinder length=0.01 radius=0.0375; visual mesh filename=meshes/center_wheel.stl
- link front_sonar: geometry collision box size=0.00001 0.00001 0.00001; visual mesh filename=meshes/front_sonar.stl
- link lms100: geometry collision box size=0.1 0.1 0.1; visual mesh filename=meshes/lms100.dae
- link p3dx_left_hubcap: geometry collision box size=0.00001 0.00001 0.00001; visual mesh filename=meshes/left_hubcap.stl
- link p3dx_left_wheel: geometry collision cylinder length=0.01 radius=0.09; visual mesh filename=meshes/left_wheel.stl
- link p3dx_right_hubcap: geometry collision box size=0.00001 0.00001 0.00001; visual mesh filename=meshes/right_hubcap.stl
- link p3dx_right_wheel: geometry collision cylinder length=0.01 radius=0.09; visual mesh filename=meshes/right_wheel.stl
- link swivel: geometry collision box size=0.00001 0.00001 0.00001; visual mesh filename=meshes/swivel.stl
- link top_plate: geometry collision box size=0.45 0.38 0.01; visual mesh filename=meshes/top.stl
