Commit message: narrow corridor test + new environment

File: system/controller/simulation/environment/obstacle_map_0/plane.urdf (robot description, URDF)
Before this commit: robot plane, 10 links, 9 joints
Links:
- removed link box_2
- removed link box_3
- removed link box_4
Joints:
- removed joint box_2_joint
- removed joint box_3_joint
- removed joint box_4_joint
