Commit message: change obstacle_map_0

File: system/controller/simulation/environment/obstacle_map_0/moveable_wall.urdf (robot description, URDF)
Before this commit: robot plane, 3 links, 2 joints
Links:
- removed link box_4
- link box_3: geometry collision box size=3.5 5 0.5; visual box size=3.5 5 0.5
Joints:
- removed joint box_4_joint

File: system/controller/simulation/environment/obstacle_map_0/plane.urdf (robot description, URDF)
Before this commit: robot plane, 7 links, 6 joints
Links:
- link wall_4: geometry collision box size=6 0.1 0.5; visual box size=6 0.1 0.5
